Commit message: Updated launch file so that it launches rviz2 and added wheels to robot

File: urdf/barista_robot_model.urdf (robot description, URDF)
Before this commit: robot box_bot, 1 links, 0 joints
Links:
- added link left_wheel; visual cylinder length=0.0206 radius=0.0352
- added link right_wheel; visual cylinder length=0.0206 radius=0.0352
Joints:
- added joint joint_left_wheel: type continuous, parent base_link, child left_wheel, origin xyz=0 0.128 -0.0775 rpy=0 0 0, axis 0 1 0, limit effort=10000 velocity=1000
- added joint joint_right_wheel: type continuous, parent base_link, child right_wheel, origin xyz=0 -0.128 -0.0775 rpy=0 0 0, axis 0 1 0, limit effort=10000 velocity=1000

Commit message: Added four standoff rods and top base to robot model

File: urdf/barista_robot_model.urdf (robot description, URDF)
Before this commit: robot box_bot, 3 links, 2 joints
Links:
- added link standoff_rod_1; visual cylinder length=0.220 radius=0.010
- added link standoff_rod_2; visual cylinder length=0.220 radius=0.010
- added link standoff_rod_3; visual cylinder length=0.220 radius=0.010
- added link standoff_rod_4; visual cylinder length=0.220 radius=0.010
- added link top_base; visual cylinder length=0.090 radius=0.160
Joints:
- added joint joint_standoff_rod_1: type fixed, parent base_link, child standoff_rod_1, origin xyz=0.100 0.100 0.1875 rpy=0 0 0
- added joint joint_standoff_rod_2: type fixed, parent base_link, child standoff_rod_2, origin xyz=-0.100 0.100 0.1875 rpy=0 0 0
- added joint joint_standoff_rod_3: type fixed, parent base_link, child standoff_rod_3, origin xyz=-0.100 -0.100 0.1875 rpy=0 0 0
- added joint joint_standoff_rod_4: type fixed, parent base_link, child standoff_rod_4, origin xyz=0.100 -0.100 0.1875 rpy=0 0 0
- added joint joint_top_base: type fixed, parent base_link, child top_base, origin xyz=0 0 0.3425 rpy=0 0 0

Commit message: Added two caster wheels

File: urdf/barista_robot_model.urdf (robot description, URDF)
Before this commit: robot box_bot, 8 links, 7 joints
Links:
- added link back_pitch_link; visual sphere radius=0.0352
- added link back_roll_link; visual cylinder length=0.0206 radius=0.0352
- added link back_yaw_link; visual cylinder length=0.0206 radius=0.0352
- added link front_pitch_link; visual sphere radius=0.0352
- added link front_roll_link; visual cylinder length=0.0206 radius=0.0352
- added link front_yaw_link; visual cylinder length=0.0206 radius=0.0352
Joints:
- added joint back_pitch_joint: type continuous, parent back_roll_link, child back_pitch_link, origin xyz=0 0 0 rpy=0 0 0, axis 0 1 0, limit effort=1000.0 velocity=100.0
- added joint back_roll_joint: type continuous, parent back_yaw_link, child back_roll_link, origin xyz=0 0 0 rpy=0 0 0, axis 1 0 0, limit effort=1000.0 velocity=100.0
- added joint back_yaw_joint: type continuous, parent base_link, child back_yaw_link, origin xyz=-0.120 0 -0.0775 rpy=0 0 0, axis 0 0 1, limit effort=1000.0 velocity=100.0
- added joint front_pitch_joint: type continuous, parent front_roll_link, child front_pitch_link, origin xyz=0 0 0 rpy=0 0 0, axis 0 1 0, limit effort=1000.0 velocity=100.0
- added joint front_roll_joint: type continuous, parent front_yaw_link, child front_roll_link, origin xyz=0 0 0 rpy=0 0 0, axis 1 0 0, limit effort=1000.0 velocity=100.0
- added joint front_yaw_joint: type continuous, parent base_link, child front_yaw_link, origin xyz=0.120 0 -0.0775 rpy=0 0 0, axis 0 0 1, limit effort=1000.0 velocity=100.0

Commit message: Added inertial and collision properties to each robot part

File: urdf/barista_robot_model.urdf (robot description, URDF)
Before this commit: robot box_bot, 14 links, 13 joints
Links:
- link back_pitch_link: mass None -> 0.05; geometry collision sphere radius=0.0352; visual sphere radius=0.0352
- link back_roll_link: mass None -> 0.001; geometry collision cylinder length=0.001 radius=0.0045000000000000005; visual cylinder length=0.001 radius=0.0045000000000000005
- link back_yaw_link: mass None -> 0.001; geometry collision cylinder length=0.001 radius=0.0045000000000000005; visual cylinder length=0.001 radius=0.0045000000000000005
- link base_link: mass None -> 2.35; geometry collision cylinder length=0.155 radius=0.178; visual cylinder length=0.155 radius=0.178
- link front_pitch_link: mass None -> 0.05; geometry collision sphere radius=0.0352; visual sphere radius=0.0352
- link front_roll_link: mass None -> 0.001; geometry collision cylinder length=0.001 radius=0.0045000000000000005; visual cylinder length=0.001 radius=0.0045000000000000005
- link front_yaw_link: mass None -> 0.001; geometry collision cylinder length=0.001 radius=0.0045000000000000005; visual cylinder length=0.001 radius=0.0045000000000000005
- link left_wheel: mass None -> 0.2; geometry collision cylinder length=0.0206 radius=0.0352; visual cylinder length=0.0206 radius=0.0352
- link right_wheel: mass None -> 0.2; geometry collision cylinder length=0.0206 radius=0.0352; visual cylinder length=0.0206 radius=0.0352
- link standoff_rod_1: mass None -> 0.05; geometry collision cylinder length=0.220 radius=0.010; visual cylinder length=0.220 radius=0.010
- link standoff_rod_2: mass None -> 0.05; geometry collision cylinder length=0.220 radius=0.010; visual cylinder length=0.220 radius=0.010
- link standoff_rod_3: mass None -> 0.05; geometry collision cylinder length=0.220 radius=0.010; visual cylinder length=0.220 radius=0.010
- link standoff_rod_4: mass None -> 0.05; geometry collision cylinder length=0.220 radius=0.010; visual cylinder length=0.220 radius=0.010
- link top_base: mass None -> 0.5; geometry collision cylinder length=0.090 radius=0.160; visual cylinder length=0.090 radius=0.160

Commit message: Added laser and tested by adding a cylinder next to the robot; laser readings appear to work correctly when I echo /scan

File: urdf/barista_robot_model.urdf (robot description, URDF)
Before this commit: robot box_bot, 14 links, 13 joints
Links:
- added link laser_scan_frame
- added link laser_scan_link, mass 0.01; collision box size=0.074986 0.074935 0.0408; visual mesh filename=package://barista_robot_description/models/hokuyo_urg_04lx.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 scale=1.0 1.0 1.0
Joints:
- added joint laser_scan_frame_joint: type fixed, parent laser_scan_link, child laser_scan_frame, origin xyz=0 0 0.03 rpy=0 0 0
- added joint laser_scan_link_joint: type fixed, parent base_link, child laser_scan_link, origin xyz=0.0 0.0 0.065 rpy=0 0 0

Commit message: Moved laser scanner to the front of the robot

File: urdf/barista_robot_model.urdf (robot description, URDF)
Before this commit: robot barista_robot, 16 links, 15 joints
Joints:
- joint laser_scan_link_joint: origin xyz=0.0 0.0 0.065 rpy=0 0 0 -> xyz=0.115 0.0 0.065 rpy=0 0 0

Commit message: Added frame name to gazebo laser scan plugin, which fixes the heigh difference between rays and laser scan object. Rays no longer at ground level in rviz

File: urdf/barista_robot_model.urdf (robot description, URDF)
Before this commit: robot barista_robot, 16 links, 15 joints
Joints:
- joint laser_scan_frame_joint: origin xyz=0 0 0.03 rpy=0 0 0 -> xyz=0 0 0.055 rpy=0 0 0

File: xacro/barista_robot_model.urdf.xacro (robot description, xacro)
@@ -376,5 +376,5 @@
         </link>
         <joint name="laser_scan_frame_joint" type="fixed">
-            <origin rpy="0 0 0" xyz="0 0 0.03"/>
+            <origin rpy="0 0 0" xyz="0 0 0.055"/>
             <parent link="laser_scan_link"/>
             <child link="laser_scan_frame"/>
@@ -402,5 +402,5 @@
             <always_on>true</always_on>
             <visualize>true</visualize>
-            <update_rate>100.0</update_rate>
+            <update_rate>30.0</update_rate>
             <plugin name="laser" filename="libgazebo_ros_ray_sensor.so">
             <ros>
@@ -409,4 +409,5 @@
             </ros>
             <output_type>sensor_msgs/LaserScan</output_type>
+            <frame_name>laser_scan_frame</frame_name>
             </plugin>
         </sensor>
