Commit message: Fixed starting position in launch file and added properties for each part of the robot

File: xacro/barista_robot_model.urdf.xacro (robot description, xacro)
@@ -1,18 +1,31 @@
 <?xml version="1.0"?>
 <robot xmlns:xacro="http://www.ros.org/wiki/xacro" name="barista_robot">
-    <material name="green_dark">
-        <color rgba="0.0 0.5 0.0 1"/>
-    </material>
-    <material name="gray">
-        <color rgba="0.5 0.5 0.5 1.0"/>
-    </material>
-    <material name="black">
-        <color rgba="0.0 0.0 0.0 1"/>
-    </material>
-    <!-- main body -->
+    <xacro:property name="base_radius" value="0.178"/>
+    <xacro:property name="base_length" value="0.155"/>
+    <xacro:property name="base_mass" value="2.35"/>
+    <xacro:property name="wheel_radius" value="0.0352"/>
+    <xacro:property name="wheel_length" value="0.0206"/>
+    <xacro:property name="wheel_mass" value="0.2"/>
+    <xacro:property name="wheel_friction" value="1.0"/>
+    <xacro:property name="wheel_damping" value="1.0"/>
+    <xacro:property name="wheel_effort_limit" value="10000"/>
+    <xacro:property name="wheel_velocity_limit" value="1000"/>
+    <xacro:property name="caster_radius" value="0.0352"/>
+    <xacro:property name="caster_mass" value="0.05"/>
+    <xacro:property name="caster_friction" value="0.1"/>
+    <xacro:property name="caster_damping" value="0.0"/>
+    <xacro:property name="caster_effort_limit" value="1000.0"/>
+    <xacro:property name="caster_velocity_limit" value="100.0"/>
+    <xacro:property name="standoff_radius" value="0.010"/>
+    <xacro:property name="standoff_length" value="0.220"/>
+    <xacro:property name="standoff_mass" value="0.05"/>
+    <xacro:property name="top_base_radius" value="0.160"/>
+    <xacro:property name="top_base_length" value="0.090"/>
+    <xacro:property name="top_base_mass" value="0.5"/>
+    <xacro:property name="top_base_z_offset" value="0.3425"/>
     <link name="base_link">
         <visual>
             <geometry>
-                <cylinder radius="0.178" length="0.155"/>
+                <cylinder radius="${base_radius}" length="${base_length}"/>
             </geometry>
             <material name="green_dark"/>
@@ -21,15 +34,364 @@
             <origin rpy="0 0 0" xyz="0 0 0"/>
             <geometry>
-                <cylinder radius="0.178" length="0.155"/>
-            </geometry>
-        </collision>
-        <inertial>
-            <origin rpy="0 0 0" xyz="0 0 0"/>
-            <mass value="2.35"/>
+                <cylinder radius="${base_radius}" length="${base_length}"/>
+            </geometry>
+        </collision>
+        <inertial>
+            <origin rpy="0 0 0" xyz="0 0 0"/>
+            <mass value="${base_mass}"/>
             <inertia ixx="0.01392573958333333" ixy="0" ixz="0" iyy="0.01392573958333333" iyz="0" izz="0.02650260416666667"/>
         </inertial>
     </link>
-    <gazebo reference="base_link">
-        <material>Gazebo/Green</material>
-    </gazebo>
+     <!-- Left Wheel -->
+    <link name="left_wheel">
+        <visual>
+            <origin rpy="0 1.5707 1.5707" xyz="0 0 0"/>
+            <geometry>
+                <cylinder length="${wheel_length}" radius="${wheel_radius}"/>
+            </geometry>
+            <material name="black"/>
+        </visual>
+        <collision>
+            <origin rpy="0 1.5707 1.5707" xyz="0 0 0"/>
+            <geometry>
+                <cylinder length="${wheel_length}" radius="${wheel_radius}"/>
+            </geometry>
+        </collision>
+        <inertial>
+            <origin rpy="0 1.5707 1.5707" xyz="0 0 0"/>
+            <mass value="${wheel_mass}"/>
+            <inertia ixx="3.07426666666667e-05" ixy="0" ixz="0" iyy="3.07426666666667e-05" iyz="0" izz="6.12266666666667e-05"/>
+        </inertial>
+    </link>
+    <joint name="joint_left_wheel" type="continuous">
+        <origin rpy="0 0 0" xyz="0 0.128 -0.0775"/>
+        <child link="left_wheel"/>
+        <parent link="base_link"/>
+        <axis rpy="0 0 0" xyz="0 1 0"/>
+        <limit effort="${wheel_effort_limit}" velocity="${wheel_velocity_limit}"/>
+        <joint_properties damping="${wheel_damping}" friction="${wheel_friction}"/>
+    </joint>
+    <!-- Right Wheel -->
+    <link name="right_wheel">
+        <visual>
+            <origin rpy="0 1.5707 1.5707" xyz="0 0 0"/>
+            <geometry>
+                <cylinder length="${wheel_length}" radius="${wheel_radius}"/>
+            </geometry>
+        </visual>
+        <collision>
+            <origin rpy="0 1.5707 1.5707" xyz="0 0 0"/>
+            <geometry>
+                <cylinder length="${wheel_length}" radius="${wheel_radius}"/>
+            </geometry>
+        </collision>
+        <inertial>
+            <origin rpy="0 1.5707 1.5707" xyz="0 0 0"/>
+            <mass value="${wheel_mass}"/>
+            <inertia ixx="3.07426666666667e-05" ixy="0" ixz="0" iyy="3.07426666666667e-05" iyz="0" izz="6.12266666666667e-05"/>
+        </inertial>
+    </link>
+    <joint name="joint_right_wheel" type="continuous">
+        <origin rpy="0 0 0" xyz="0 -0.128 -0.0775"/>
+        <child link="right_wheel"/>
+        <parent link="base_link"/>
+        <axis rpy="0 0 0" xyz="0 1 0"/>
+        <limit effort="${wheel_effort_limit}" velocity="${wheel_velocity_limit}"/>
+        <joint_properties damping="${wheel_damping}" friction="${wheel_friction}"/>
+    </joint>
+    <!-- Caster Wheel Front -->
+    <link name="front_yaw_link">
+    <visual>
+        <origin rpy="0 1.5707 1.5707" xyz="0 0 0"/>
+        <geometry>
+        <cylinder length="0.001" radius="0.0045000000000000005"/>
+        </geometry>
+        <material name="gray"/>
+    </visual>
+    <collision>
+        <origin rpy="0 1.5707 1.5707" xyz="0 0 0"/>
+        <geometry>
+        <cylinder length="0.001" radius="0.0045000000000000005"/>
+        </geometry>
+    </collision>
+    <inertial>
+        <origin rpy="0 1.5707 1.5707" xyz="0 0 0"/>
+        <mass value="0.001"/>
+        <inertia ixx="5.145833333333334e-09" ixy="0" ixz="0" iyy="5.145833333333334e-09" iyz="0" izz="1.0125000000000003e-08"/>
+    </inertial>
+    </link>
+    <joint name="front_yaw_joint" type="continuous">
+    <origin rpy="0 0 0" xyz="0.120 0 -0.0775" />
+    <parent link="base_link" />
+    <child link="front_yaw_link" />
+    <axis xyz="0 0 1" />
+    <limit effort="${caster_effort_limit}" velocity="${caster_velocity_limit}" />
+    <dynamics damping="${caster_damping}" friction="${caster_friction}"/>
+    </joint>
+    <link name="front_roll_link">
+    <visual>
+        <origin rpy="0 1.5707 1.5707" xyz="0 0 0"/>
+        <geometry>
+        <cylinder length="0.001" radius="0.0045000000000000005"/>
+        </geometry>
+        <material name="gray"/>
+    </visual>
+    <collision>
+        <origin rpy="0 1.5707 1.5707" xyz="0 0 0"/>
+        <geometry>
+        <cylinder length="0.001" radius="0.0045000000000000005"/>
+        </geometry>
+    </collision>
+    <inertial>
+        <origin rpy="0 1.5707 1.5707" xyz="0 0 0"/>
+        <mass value="0.001"/>
+        <inertia ixx="5.145833333333334e-09" ixy="0" ixz="0" iyy="5.145833333333334e-09" iyz="0" izz="1.0125000000000003e-08"/>
+    </inertial>
+    </link>
+    <joint name="front_roll_joint" type="continuous">
+    <origin rpy="0 0 0" xyz="0 0 0" />
+    <parent link="front_yaw_link" />
+    <child link="front_roll_link" />
+    <axis xyz="1 0 0" />
+    <limit effort="${caster_effort_limit}" velocity="${caster_velocity_limit}" />
+    <dynamics damping="${caster_damping}" friction="${caster_friction}"/>
+    </joint>
+    <link name="front_pitch_link">
+    <visual>
+        <origin rpy="0 1.5707 1.5707" xyz="0 0 0"/>
+        <geometry>
+        <sphere radius="${caster_radius}"/>
+        </geometry>
+        <material name="gray"/>
+    </visual>
+    <collision>
+        <origin rpy="0 1.5707 1.5707" xyz="0 0 0"/>
+        <geometry>
+        <sphere radius="${caster_radius}"/>
+        </geometry>
+    </collision>
+    <inertial>
+        <origin rpy="0 1.5707 1.5707" xyz="0 0 0"/>
+        <mass value="${caster_mass}"/>
+        <inertia ixx="1.531733333333333e-05" ixy="0" ixz="0" iyy="1.531733333333333e-05" iyz="0" izz="1.531733333333333e-05"/>
+    </inertial>
+    </link>
+    <joint name="front_pitch_joint" type="continuous">
+    <origin rpy="0 0 0" xyz="0 0 0" />
+    <parent link="front_roll_link" />
+    <child link="front_pitch_link" />
+    <axis xyz="0 1 0" />
+    <limit effort="${caster_effort_limit}" velocity="${caster_velocity_limit}" />
+    <dynamics damping="${caster_damping}" friction="${caster_friction}"/>
+    </joint>
+    <!-- Caster Wheel Back -->
+    <link name="back_yaw_link">
+    <visual>
+        <origin rpy="0 1.5707 1.5707" xyz="0 0 0"/>
+        <geometry>
+        <cylinder length="0.001" radius="0.0045000000000000005"/>
+        </geometry>
+        <material name="gray"/>
+    </visual>
+    <collision>
+        <origin rpy="0 1.5707 1.5707" xyz="0 0 0"/>
+        <geometry>
+        <cylinder length="0.001" radius="0.0045000000000000005"/>
+        </geometry>
+    </collision>
+    <inertial>
+        <origin rpy="0 1.5707 1.5707" xyz="0 0 0"/>
+        <mass value="0.001"/>
+        <inertia ixx="5.145833333333334e-09" ixy="0" ixz="0" iyy="5.145833333333334e-09" iyz="0" izz="1.0125000000000003e-08"/>
+    </inertial>
+    </link>
+    <joint name="back_yaw_joint" type="continuous">
+    <origin rpy="0 0 0" xyz="-0.120 0 -0.0775" />
+    <parent link="base_link" />
+    <child link="back_yaw_link" />
+    <axis xyz="0 0 1" />
+    <limit effort="${caster_effort_limit}" velocity="${caster_velocity_limit}" />
+    <dynamics damping="${caster_damping}" friction="${caster_friction}"/>
+    </joint>
+    <link name="back_roll_link">
+    <visual>
+        <origin rpy="0 1.5707 1.5707" xyz="0 0 0"/>
+        <geometry>
+        <cylinder length="0.001" radius="0.0045000000000000005"/>
+        </geometry>
+        <material name="gray"/>
+    </visual>
+    <collision>
+        <origin rpy="0 1.5707 1.5707" xyz="0 0 0"/>
+        <geometry>
+        <cylinder length="0.001" radius="0.0045000000000000005"/>
+        </geometry>
+    </collision>
+    <inertial>
+        <origin rpy="0 1.5707 1.5707" xyz="0 0 0"/>
+        <mass value="0.001"/>
+        <inertia ixx="5.145833333333334e-09" ixy="0" ixz="0" iyy="5.145833333333334e-09" iyz="0" izz="1.0125000000000003e-08"/>
+    </inertial>
+    </link>
+    <joint name="back_roll_joint" type="continuous">
+    <origin rpy="0 0 0" xyz="0 0 0" />
+    <parent link="back_yaw_link" />
+    <child link="back_roll_link" />
+    <axis xyz="1 0 0" />
+    <limit effort="${caster_effort_limit}" velocity="${caster_velocity_limit}" />
+    <dynamics damping="${caster_damping}" friction="${caster_friction}"/>
+    </joint>
+    <link name="back_pitch_link">
+    <visual>
+        <origin rpy="0 1.5707 1.5707" xyz="0 0 0"/>
+        <geometry>
+        <sphere radius="${caster_radius}"/>
+        </geometry>
+        <material name="gray"/>
+    </visual>
+    <collision>
+        <origin rpy="0 1.5707 1.5707" xyz="0 0 0"/>
+        <geometry>
+        <sphere radius="${caster_radius}"/>
+        </geometry>
+    </collision>
+    <inertial>
+        <origin rpy="0 1.5707 1.5707" xyz="0 0 0"/>
+        <mass value="${caster_mass}"/>
+        <inertia ixx="1.531733333333333e-05" ixy="0" ixz="0" iyy="1.531733333333333e-05" iyz="0" izz="1.531733333333333e-05"/>
+    </inertial>
+    </link>
+    <joint name="back_pitch_joint" type="continuous">
+    <origin rpy="0 0 0" xyz="0 0 0" />
+    <parent link="back_roll_link" />
+    <child link="back_pitch_link" />
+    <axis xyz="0 1 0" />
+    <limit effort="${caster_effort_limit}" velocity="${caster_velocity_limit}" />
+    <dynamics damping="${caster_damping}" friction="${caster_friction}"/>
+    </joint>
+   <!-- Standoff Rod 1 -->
+    <link name="standoff_rod_1">
+        <visual>
+            <origin rpy="0 0 0" xyz="0 0 0"/>
+            <geometry>
+            <cylinder length="${standoff_length}" radius="${standoff_radius}"/>
+            </geometry>
+        </visual>
+        <collision>
+            <origin rpy="0 0 0" xyz="0 0 0"/>
+            <geometry>
+            <cylinder length="${standoff_length}" radius="${standoff_radius}"/>
+            </geometry>
+        </collision>
+        <inertial>
+            <origin rpy="0 0 0" xyz="0 0 0"/>
+            <mass value="${standoff_mass}"/>
+            <inertia ixx="2.058333333333333e-06" ixy="0" ixz="0" iyy="2.058333333333333e-06" iyz="0" izz="5.0625e-09"/>
+        </inertial>
+    </link>
+    <joint name="joint_standoff_rod_1" type="fixed">
+        <origin rpy="0 0 0" xyz="0.100 0.100 0.1875"/>
+        <parent link="base_link"/>
+        <child link="standoff_rod_1"/>
+    </joint>
+    <!-- Standoff Rod 2 -->
+    <link name="standoff_rod_2">
+        <visual>
+            <origin rpy="0 0 0" xyz="0 0 0"/>
+            <geometry>
+            <cylinder length="${standoff_length}" radius="${standoff_radius}"/>
+            </geometry>
+        </visual>
+        <collision>
+            <origin rpy="0 0 0" xyz="0 0 0"/>
+            <geometry>
+            <cylinder length="${standoff_length}" radius="${standoff_radius}"/>
+            </geometry>
+        </collision>
+        <inertial>
+            <origin rpy="0 0 0" xyz="0 0 0"/>
+            <mass value="${standoff_mass}"/>
+            <inertia ixx="2.058333333333333e-06" ixy="0" ixz="0" iyy="2.058333333333333e-06" iyz="0" izz="5.0625e-09"/>
+        </inertial>
+    </link>
+    <joint name="joint_standoff_rod_2" type="fixed">
+        <origin rpy="0 0 0" xyz="-0.100 0.100 0.1875"/>
+        <parent link="base_link"/>
+        <child link="standoff_rod_2"/>
+    </joint>
+    <!-- Standoff Rod 3 -->
+    <link name="standoff_rod_3">
+        <visual>
+            <origin rpy="0 0 0" xyz="0 0 0"/>
+            <geometry>
+            <cylinder length="${standoff_length}" radius="${standoff_radius}"/>
+            </geometry>
+        </visual>
+        <collision>
+            <origin rpy="0 0 0" xyz="0 0 0"/>
+            <geometry>
+            <cylinder length="${standoff_length}" radius="${standoff_radius}"/>
+            </geometry>
+        </collision>
+        <inertial>
+            <origin rpy="0 0 0" xyz="0 0 0"/>
+            <mass value="${standoff_mass}"/>
+            <inertia ixx="2.058333333333333e-06" ixy="0" ixz="0" iyy="2.058333333333333e-06" iyz="0" izz="5.0625e-09"/>
+        </inertial>
+    </link>
+    <joint name="joint_standoff_rod_3" type="fixed">
+        <origin rpy="0 0 0" xyz="-0.100 -0.100 0.1875"/>
+        <parent link="base_link"/>
+        <child link="standoff_rod_3"/>
+    </joint>
+    <!-- Standoff Rod 4 -->
+    <link name="standoff_rod_4">
+        <visual>
+            <origin rpy="0 0 0" xyz="0 0 0"/>
+            <geometry>
+            <cylinder length="${standoff_length}" radius="${standoff_radius}"/>
+            </geometry>
+        </visual>
+        <collision>
+            <origin rpy="0 0 0" xyz="0 0 0"/>
+            <geometry>
+            <cylinder length="${standoff_length}" radius="${standoff_radius}"/>
+            </geometry>
+        </collision>
+        <inertial>
+            <origin rpy="0 0 0" xyz="0 0 0"/>
+            <mass value="${standoff_mass}"/>
+            <inertia ixx="2.058333333333333e-06" ixy="0" ixz="0" iyy="2.058333333333333e-06" iyz="0" izz="5.0625e-09"/>
+        </inertial>
+    </link>
+    <joint name="joint_standoff_rod_4" type="fixed">
+        <origin rpy="0 0 0" xyz="0.100 -0.100 0.1875"/>
+        <parent link="base_link"/>
+        <child link="standoff_rod_4"/>
+    </joint>
+    <!-- Top Base -->
+    <link name="top_base">
+    <visual>
+        <geometry>
+        <cylinder radius="${top_base_radius}" length="${top_base_length}"/>
+        </geometry>
+        <material name="green_dark"/>
+    </visual>
+    <collision>
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