Commit message: Added gazebo related tags into xacro file and updated launch file

File: xacro/barista_robot_model.urdf.xacro (robot description, xacro)
@@ -27,4 +27,5 @@
     <xacro:property name="top_base_mass" value="0.5"/>
     <xacro:property name="top_base_z_offset" value="0.3425"/>
+    <xacro:property name="include_laser" value="true"/>
     <link name="base_link">
         <visual>
@@ -46,6 +47,36 @@
         </inertial>
     </link>
-    <xacro:wheel wheel_name="left_wheel" wheel_position="0.128" />
-    <xacro:wheel wheel_name="right_wheel" wheel_position="-0.128" />
+    <xacro:wheel wheel_name="left_wheel" />
+    <xacro:wheel wheel_name="right_wheel" />
+    <gazebo reference="left_wheel">
+        <kp>1000000000000000000000000000.0</kp>
+        <kd>1000000000000000000000000000.0</kd>
+        <mu1>10.0</mu1>
+        <mu2>10.0</mu2>
+        <material>Gazebo/Black</material>
+    </gazebo>
+    <joint name="joint_left_wheel" type="continuous">
+        <origin rpy="0 0 0" xyz="0 0.128 -0.0775"/>
+        <child link="left_wheel"/>
+        <parent link="base_link"/>
+        <axis rpy="0 0 0" xyz="0 1 0"/>
+        <limit effort="10000" velocity="1000"/>
+        <joint_properties damping="1.0" friction="1.0"/>
+    </joint>
+    <gazebo reference="right_wheel">
+        <kp>1000000000000000000000000000.0</kp>
+        <kd>1000000000000000000000000000.0</kd>
+        <mu1>10.0</mu1>
+        <mu2>10.0</mu2>
+        <material>Gazebo/Black</material>
+    </gazebo>
+    <joint name="joint_right_wheel" type="continuous">
+        <origin rpy="0 0 0" xyz="0 -0.128 -0.0775"/>
+        <child link="right_wheel"/>
+        <parent link="base_link"/>
+        <axis rpy="0 0 0" xyz="0 1 0"/>
+        <limit effort="10000" velocity="1000"/>
+        <joint_properties damping="1.0" friction="1.0"/>
+    </joint>
     <!-- Caster Wheel Front -->
     <link name="front_yaw_link">
@@ -125,4 +156,11 @@
     </inertial>
     </link>
+    <gazebo reference="front_pitch_link">
+        <kp>1000000000000000000000000000.0</kp>
+        <kd>1000000000000000000000000000.0</kd>
+        <mu1>0.5</mu1>
+        <mu2>0.5</mu2>
+        <material>Gazebo/Grey</material>
+    </gazebo>
     <joint name="front_pitch_joint" type="continuous">
     <origin rpy="0 0 0" xyz="0 0 0" />
@@ -210,4 +248,11 @@
     </inertial>
     </link>
+    <gazebo reference="back_pitch_link">
+        <kp>1000000000000000000000000000.0</kp>
+        <kd>1000000000000000000000000000.0</kd>
+        <mu1>0.5</mu1>
+        <mu2>0.5</mu2>
+        <material>Gazebo/Grey</material>
+    </gazebo>
     <joint name="back_pitch_joint" type="continuous">
     <origin rpy="0 0 0" xyz="0 0 0" />
@@ -218,9 +263,152 @@
     <dynamics damping="${caster_damping}" friction="${caster_friction}"/>
     </joint>
-    <xacro:standoff_rod rod_name="standoff_rod_1" rod_x_pos="0.100" rod_y_pos="0.100" />
-    <xacro:standoff_rod rod_name="standoff_rod_2" rod_x_pos="-0.100" rod_y_pos="0.100" />
-    <xacro:standoff_rod rod_name="standoff_rod_3" rod_x_pos="-0.100" rod_y_pos="-0.100" />
-    <xacro:standoff_rod rod_name="standoff_rod_4" rod_x_pos="0.100" rod_y_pos="-0.100" />
+    <xacro:standoff_rod rod_name="standoff_rod_1" />
+    <xacro:standoff_rod rod_name="standoff_rod_2" />
+    <xacro:standoff_rod rod_name="standoff_rod_3" />
+    <xacro:standoff_rod rod_name="standoff_rod_4" />
+    <gazebo reference="standoff_rod_1">
+        <material>Gazebo/Grey</material>
+    </gazebo>
+    <joint name="joint_standoff_rod_1" type="fixed">
+        <origin rpy="0 0 0" xyz="0.100 0.100 0.1875"/>
+        <parent link="base_link"/>
+        <child link="standoff_rod_1"/>
+    </joint>
+    <gazebo reference="standoff_rod_2">
+        <material>Gazebo/Grey</material>
+    </gazebo>
+    <joint name="joint_standoff_rod_2" type="fixed">
+        <origin rpy="0 0 0" xyz="-0.100 0.100 0.1875"/>
+        <parent link="base_link"/>
+        <child link="standoff_rod_2"/>
+    </joint>
+    <gazebo reference="standoff_rod_3">
+        <material>Gazebo/Grey</material>
+    </gazebo>
+    <joint name="joint_standoff_rod_3" type="fixed">
+        <origin rpy="0 0 0" xyz="-0.100 -0.100 0.1875"/>
+        <parent link="base_link"/>
+        <child link="standoff_rod_3"/>
+    </joint>
+    <gazebo reference="standoff_rod_4">
+        <material>Gazebo/Grey</material>
+    </gazebo>
+    <joint name="joint_standoff_rod_4" type="fixed">
+        <origin rpy="0 0 0" xyz="0.100 -0.100 0.1875"/>
+        <parent link="base_link"/>
+        <child link="standoff_rod_4"/>
+    </joint>
     <!-- Top Base -->
     <xacro:cup_holder_tray tray_z_pos="${top_base_z_offset}" />
+    <gazebo reference="top_base">
+        <material>Gazebo/Green</material>
+    </gazebo>
+    <joint name="joint_top_base" type="fixed">
+        <origin rpy="0 0 0" xyz="0 0 0.3425"/>
+        <parent link="base_link"/>
+        <child link="top_base"/>
+    </joint>
+    <!-- PLUGINS -->
+    <!-- JOINT PUBLISHER -->
+    <gazebo>
+        <plugin name="box_bot_joint_state" filename="libgazebo_ros_joint_state_publisher.so">
+        <ros>
+            <remapping>~/out:=joint_states</remapping>
+        </ros>
+        <update_rate>30</update_rate>
+        <joint_name>joint_left_wheel</joint_name>
+        <joint_name>joint_right_wheel</joint_name>
+        <joint_name>front_yaw_joint</joint_name>
+        <joint_name>back_yaw_joint</joint_name>
+        <joint_name>front_roll_joint</joint_name>
+        <joint_name>back_roll_joint</joint_name>
+        <joint_name>front_pitch_joint</joint_name>
+        <joint_name>back_pitch_joint</joint_name>
+        </plugin>
+    </gazebo>
+    <!-- Differential drive -->
+    <gazebo>
+        <plugin filename="libgazebo_ros_diff_drive.so" name="differential_drive_controller">
+        <!-- wheels -->
+        <left_joint>joint_left_wheel</left_joint>
+        <right_joint>joint_right_wheel</right_joint>
+        <!-- kinematics -->
+        <wheel_separation>0.1</wheel_separation>
+        <wheel_diameter>0.07</wheel_diameter>
+        <!-- limits -->
+        <max_wheel_torque>1.0</max_wheel_torque>
+        <max_wheel_acceleration>2.0</max_wheel_acceleration>
+        <!-- output -->
+        <publish_odom>true</publish_odom>
+        <publish_odom_tf>true</publish_odom_tf>
+        <odometry_frame>odom</odometry_frame>
+        <robot_base_frame>base_link</robot_base_frame>
+        </plugin>
+  </gazebo>
+    <!-- Laser Scanner -->
+    <xacro:macro name="laser_scanner" params="include_laser">
+        <xacro:if value="${include_laser}">
+        <link name="laser_scan_link">
+            <visual>
+            <origin rpy="0 0 0" xyz="0 0 0"/>
+            <geometry>
+                <mesh filename="package://barista_robot_description/models/hokuyo_urg_04lx.dae" scale="1.0 1.0 1.0"/>
+            </geometry>
+            </visual>
+            <collision>
+            <origin rpy="0 0 0" xyz="0 0 0.0204"/>
+            <geometry>
+                <box size="0.074986 0.074935 0.0408"/>
+            </geometry>
+            </collision>
+            <inertial>
+            <mass value="0.01"/>
+            <origin rpy="0 0 0" xyz="0 0 0.0204"/>
+            <inertia ixx="6.066578520833334e-06" ixy="0" ixz="0" iyy="6.072950163333333e-06" iyz="0" izz="9.365128684166666e-06"/>
+            </inertial>
+        </link>
+        <joint name="laser_scan_link_joint" type="fixed">
+            <origin rpy="0 0 0" xyz="0.0 0.0 0.065"/>
+            <parent link="cup_holder_tray"/>
+            <child link="laser_scan_link"/>
+        </joint>
+        <link name="laser_scan_frame">
+        </link>
+        <joint name="laser_scan_frame_joint" type="fixed">
+            <origin rpy="0 0 0" xyz="0 0 0.03"/>
+            <parent link="laser_scan_link"/>
+            <child link="laser_scan_frame"/>
+        </joint>
+        </xacro:if>
+    </xacro:macro>
+    <xacro:laser_scanner include_laser="${include_laser}" />
+    <gazebo reference="laser_scan_frame">
+        <sensor name="sensor_ray" type="ray">
+            <pose>0 0 0 0 0 0</pose>
+            <ray>
+            <scan>
+                <horizontal>
+                <samples>200</samples>
+                <resolution>1.0</resolution>
+                <min_angle>-3.14</min_angle>
+                <max_angle>3.14</max_angle>
+                </horizontal>
+            </scan>
+            <range>
+                <min>0.1</min>
+                <max>5.0</max>
+            </range>
+            </ray>
+            <always_on>true</always_on>
+            <visualize>true</visualize>
+            <update_rate>100.0</update_rate>
+            <plugin name="laser" filename="libgazebo_ros_ray_sensor.so">
+            <ros>
+                <namespace></namespace>
+                <remapping>~/out:=scan</remapping>
+            </ros>
+            <output_type>sensor_msgs/LaserScan</output_type>
+            </plugin>
+        </sensor>
+    </gazebo>
 </robot>

File: xacro/cup_holder_tray.xacro (robot description, xacro)
@@ -21,9 +21,4 @@
             </inertial>
         </link>
-        <joint name="joint_cup_holder_tray" type="fixed">
-            <origin rpy="0 0 0" xyz="0 0 ${tray_z_pos}"/>
-            <parent link="base_link"/>
-            <child link="cup_holder_tray"/>
-        </joint>
     </xacro:macro>
 </robot>

File: xacro/standoff.xacro (robot description, xacro)
@@ -1,5 +1,5 @@
 <?xml version="1.0"?>
 <robot xmlns:xacro="http://www.ros.org/wiki/xacro" name="barista_robot">
-    <xacro:macro name="standoff_rod" params="rod_name rod_x_pos rod_y_pos">
+    <xacro:macro name="standoff_rod" params="rod_name">
         <link name="${rod_name}">
             <visual>
@@ -22,9 +22,4 @@
             </inertial>
         </link>
-        <joint name="joint_${rod_name}" type="fixed">
-            <origin rpy="0 0 0" xyz="${rod_x_pos} ${rod_y_pos} 0.1875"/>
-            <parent link="base_link"/>
-            <child link="${rod_name}"/>
-        </joint>
     </xacro:macro>
 </robot>

File: xacro/wheel.xacro (robot description, xacro)
@@ -1,5 +1,5 @@
 <?xml version="1.0"?>
 <robot xmlns:xacro="http://www.ros.org/wiki/xacro" name="barista_robot">
-    <xacro:macro name="wheel" params="wheel_name wheel_position">
+    <xacro:macro name="wheel" params="wheel_name">
         <link name="${wheel_name}">
             <visual>
@@ -22,12 +22,4 @@
             </inertial>
         </link>
-        <joint name="joint_${wheel_name}" type="continuous">
-            <origin rpy="0 0 0" xyz="0 ${wheel_position} -0.0775"/>
-            <child link="${wheel_name}"/>
-            <parent link="base_link"/>
-            <axis rpy="0 0 0" xyz="0 1 0"/>
-            <limit effort="${wheel_effort_limit}" velocity="${wheel_velocity_limit}"/>
-            <joint_properties damping="${wheel_damping}" friction="${wheel_friction}"/>
-        </joint>
     </xacro:macro>
 </robot>
