Commit message: Fixed single xacro robot launch; macros were causing errors on launch, got rid of inconsistencies in the cup_holder_tray, extracted gazebo tags to gazebo_elements macro, fixed launch file

File: xacro/barista_robot_model.urdf.xacro (robot description, xacro)
@@ -1,4 +1,5 @@
 <?xml version="1.0"?>
 <robot xmlns:xacro="http://www.ros.org/wiki/xacro" name="barista_robot">
+    <xacro:include filename="$(find barista_robot_description)/xacro/barista_robot.gazebo.xacro" />
     <xacro:include filename="$(find barista_robot_description)/xacro/wheel.xacro" />
     <xacro:include filename="$(find barista_robot_description)/xacro/standoff.xacro" />
@@ -23,9 +24,19 @@
     <xacro:property name="standoff_length" value="0.220"/>
     <xacro:property name="standoff_mass" value="0.05"/>
-    <xacro:property name="top_base_radius" value="0.160"/>
-    <xacro:property name="top_base_length" value="0.090"/>
-    <xacro:property name="top_base_mass" value="0.5"/>
-    <xacro:property name="top_base_z_offset" value="0.3425"/>
+    <xacro:property name="cup_holder_tray_radius" value="0.160"/>
+    <xacro:property name="cup_holder_tray_length" value="0.090"/>
+    <xacro:property name="cup_holder_tray_mass" value="0.5"/>
+    <xacro:property name="cup_holder_tray_z_offset" value="0.3425"/>
     <xacro:property name="include_laser" value="true"/>
+    <material name="green_dark">
+        <color rgba="0.0 0.5 0.0 1"/>
+    </material>
+    <material name="gray">
+        <color rgba="0.5 0.5 0.5 1.0"/>
+    </material>
+    <material name="black">
+        <color rgba="0.0 0.0 0.0 1"/>
+    </material>
+    <!-- main body -->
     <link name="base_link">
         <visual>
@@ -47,13 +58,6 @@
         </inertial>
     </link>
+    <!-- Left Wheel -->
     <xacro:wheel wheel_name="left_wheel" />
-    <xacro:wheel wheel_name="right_wheel" />
-    <gazebo reference="left_wheel">
-        <kp>1000000000000000000000000000.0</kp>
-        <kd>1000000000000000000000000000.0</kd>
-        <mu1>10.0</mu1>
-        <mu2>10.0</mu2>
-        <material>Gazebo/Black</material>
-    </gazebo>
     <joint name="joint_left_wheel" type="continuous">
         <origin rpy="0 0 0" xyz="0 0.128 -0.0775"/>
@@ -64,11 +68,6 @@
         <joint_properties damping="1.0" friction="1.0"/>
     </joint>
-    <gazebo reference="right_wheel">
-        <kp>1000000000000000000000000000.0</kp>
-        <kd>1000000000000000000000000000.0</kd>
-        <mu1>10.0</mu1>
-        <mu2>10.0</mu2>
-        <material>Gazebo/Black</material>
-    </gazebo>
+    <!-- Right Wheel -->
+    <xacro:wheel wheel_name="right_wheel" />
     <joint name="joint_right_wheel" type="continuous">
         <origin rpy="0 0 0" xyz="0 -0.128 -0.0775"/>
@@ -81,193 +80,174 @@
     <!-- Caster Wheel Front -->
     <link name="front_yaw_link">
-    <visual>
-        <origin rpy="0 1.5707 1.5707" xyz="0 0 0"/>
-        <geometry>
-        <cylinder length="0.001" radius="0.0045000000000000005"/>
-        </geometry>
-        <material name="gray"/>
-    </visual>
-    <collision>
-        <origin rpy="0 1.5707 1.5707" xyz="0 0 0"/>
-        <geometry>
-        <cylinder length="0.001" radius="0.0045000000000000005"/>
-        </geometry>
-    </collision>
-    <inertial>
-        <origin rpy="0 1.5707 1.5707" xyz="0 0 0"/>
-        <mass value="0.001"/>
-        <inertia ixx="5.145833333333334e-09" ixy="0" ixz="0" iyy="5.145833333333334e-09" iyz="0" izz="1.0125000000000003e-08"/>
-    </inertial>
+        <visual>
+            <origin rpy="0 1.5707 1.5707" xyz="0 0 0"/>
+            <geometry>
+            <cylinder length="0.001" radius="0.0045000000000000005"/>
+            </geometry>
+            <material name="gray"/>
+        </visual>
+        <collision>
+            <origin rpy="0 1.5707 1.5707" xyz="0 0 0"/>
+            <geometry>
+            <cylinder length="0.001" radius="0.0045000000000000005"/>
+            </geometry>
+        </collision>
+        <inertial>
+            <origin rpy="0 1.5707 1.5707" xyz="0 0 0"/>
+            <mass value="0.001"/>
+            <inertia ixx="5.145833333333334e-09" ixy="0" ixz="0" iyy="5.145833333333334e-09" iyz="0" izz="1.0125000000000003e-08"/>
+        </inertial>
     </link>
     <joint name="front_yaw_joint" type="continuous">
-    <origin rpy="0 0 0" xyz="0.120 0 -0.0775" />
-    <parent link="base_link" />
-    <child link="front_yaw_link" />
-    <axis xyz="0 0 1" />
-    <limit effort="${caster_effort_limit}" velocity="${caster_velocity_limit}" />
-    <dynamics damping="${caster_damping}" friction="${caster_friction}"/>
+        <origin rpy="0 0 0" xyz="0.120 0 -0.0775" />
+        <parent link="base_link" />
+        <child link="front_yaw_link" />
+        <axis xyz="0 0 1" />
+        <limit effort="${caster_effort_limit}" velocity="${caster_velocity_limit}" />
+        <dynamics damping="${caster_damping}" friction="${caster_friction}"/>
     </joint>
     <link name="front_roll_link">
-    <visual>
-        <origin rpy="0 1.5707 1.5707" xyz="0 0 0"/>
-        <geometry>
-        <cylinder length="0.001" radius="0.0045000000000000005"/>
-        </geometry>
-        <material name="gray"/>
-    </visual>
-    <collision>
-        <origin rpy="0 1.5707 1.5707" xyz="0 0 0"/>
-        <geometry>
-        <cylinder length="0.001" radius="0.0045000000000000005"/>
-        </geometry>
-    </collision>
-    <inertial>
-        <origin rpy="0 1.5707 1.5707" xyz="0 0 0"/>
-        <mass value="0.001"/>
-        <inertia ixx="5.145833333333334e-09" ixy="0" ixz="0" iyy="5.145833333333334e-09" iyz="0" izz="1.0125000000000003e-08"/>
-    </inertial>
+        <visual>
+            <origin rpy="0 1.5707 1.5707" xyz="0 0 0"/>
+            <geometry>
+            <cylinder length="0.001" radius="0.0045000000000000005"/>
+            </geometry>
+            <material name="gray"/>
+        </visual>
+        <collision>
+            <origin rpy="0 1.5707 1.5707" xyz="0 0 0"/>
+            <geometry>
+            <cylinder length="0.001" radius="0.0045000000000000005"/>
+            </geometry>
+        </collision>
+        <inertial>
+            <origin rpy="0 1.5707 1.5707" xyz="0 0 0"/>
+            <mass value="0.001"/>
+            <inertia ixx="5.145833333333334e-09" ixy="0" ixz="0" iyy="5.145833333333334e-09" iyz="0" izz="1.0125000000000003e-08"/>
+        </inertial>
     </link>
     <joint name="front_roll_joint" type="continuous">
-    <origin rpy="0 0 0" xyz="0 0 0" />
-    <parent link="front_yaw_link" />
-    <child link="front_roll_link" />
-    <axis xyz="1 0 0" />
-    <limit effort="${caster_effort_limit}" velocity="${caster_velocity_limit}" />
-    <dynamics damping="${caster_damping}" friction="${caster_friction}"/>
+        <origin rpy="0 0 0" xyz="0 0 0" />
+        <parent link="front_yaw_link" />
+        <child link="front_roll_link" />
+        <axis xyz="1 0 0" />
+        <limit effort="${caster_effort_limit}" velocity="${caster_velocity_limit}" />
+        <dynamics damping="${caster_damping}" friction="${caster_friction}"/>
     </joint>
     <link name="front_pitch_link">
-    <visual>
-        <origin rpy="0 1.5707 1.5707" xyz="0 0 0"/>
-        <geometry>
-        <sphere radius="${caster_radius}"/>
-        </geometry>
-        <material name="gray"/>
-    </visual>
-    <collision>
-        <origin rpy="0 1.5707 1.5707" xyz="0 0 0"/>
-        <geometry>
-        <sphere radius="${caster_radius}"/>
-        </geometry>
-    </collision>
-    <inertial>
-        <origin rpy="0 1.5707 1.5707" xyz="0 0 0"/>
-        <mass value="${caster_mass}"/>
-        <inertia ixx="1.531733333333333e-05" ixy="0" ixz="0" iyy="1.531733333333333e-05" iyz="0" izz="1.531733333333333e-05"/>
-    </inertial>
-    </link>
-    <gazebo reference="front_pitch_link">
-        <kp>1000000000000000000000000000.0</kp>
-        <kd>1000000000000000000000000000.0</kd>
-        <mu1>0.5</mu1>
-        <mu2>0.5</mu2>
-        <material>Gazebo/Grey</material>
-    </gazebo>
+        <visual>
+            <origin rpy="0 1.5707 1.5707" xyz="0 0 0"/>
+            <geometry>
+            <sphere radius="${caster_radius}"/>
+            </geometry>
+            <material name="gray"/>
+        </visual>
+        <collision>
+            <origin rpy="0 1.5707 1.5707" xyz="0 0 0"/>
+            <geometry>
+            <sphere radius="${caster_radius}"/>
+            </geometry>
+        </collision>
+        <inertial>
+            <origin rpy="0 1.5707 1.5707" xyz="0 0 0"/>
+            <mass value="${caster_mass}"/>
+            <inertia ixx="1.531733333333333e-05" ixy="0" ixz="0" iyy="1.531733333333333e-05" iyz="0" izz="1.531733333333333e-05"/>
+        </inertial>
+    </link>
     <joint name="front_pitch_joint" type="continuous">
-    <origin rpy="0 0 0" xyz="0 0 0" />
-    <parent link="front_roll_link" />
-    <child link="front_pitch_link" />
-    <axis xyz="0 1 0" />
-    <limit effort="${caster_effort_limit}" velocity="${caster_velocity_limit}" />
-    <dynamics damping="${caster_damping}" friction="${caster_friction}"/>
+        <origin rpy="0 0 0" xyz="0 0 0" />
+        <parent link="front_roll_link" />
+        <child link="front_pitch_link" />
+        <axis xyz="0 1 0" />
+        <limit effort="${caster_effort_limit}" velocity="${caster_velocity_limit}" />
+        <dynamics damping="${caster_damping}" friction="${caster_friction}"/>
     </joint>
     <!-- Caster Wheel Back -->
     <link name="back_yaw_link">
-    <visual>
-        <origin rpy="0 1.5707 1.5707" xyz="0 0 0"/>
-        <geometry>
-        <cylinder length="0.001" radius="0.0045000000000000005"/>
-        </geometry>
-        <material name="gray"/>
-    </visual>
-    <collision>
-        <origin rpy="0 1.5707 1.5707" xyz="0 0 0"/>
-        <geometry>
-        <cylinder length="0.001" radius="0.0045000000000000005"/>
-        </geometry>
-    </collision>
-    <inertial>
-        <origin rpy="0 1.5707 1.5707" xyz="0 0 0"/>
-        <mass value="0.001"/>
-        <inertia ixx="5.145833333333334e-09" ixy="0" ixz="0" iyy="5.145833333333334e-09" iyz="0" izz="1.0125000000000003e-08"/>
-    </inertial>
+        <visual>
+            <origin rpy="0 1.5707 1.5707" xyz="0 0 0"/>
+            <geometry>
+            <cylinder length="0.001" radius="0.0045000000000000005"/>
+            </geometry>
+            <material name="gray"/>
+        </visual>
+        <collision>
+            <origin rpy="0 1.5707 1.5707" xyz="0 0 0"/>
+            <geometry>
+            <cylinder length="0.001" radius="0.0045000000000000005"/>
+            </geometry>
+        </collision>
+        <inertial>
+            <origin rpy="0 1.5707 1.5707" xyz="0 0 0"/>
+            <mass value="0.001"/>
+            <inertia ixx="5.145833333333334e-09" ixy="0" ixz="0" iyy="5.145833333333334e-09" iyz="0" izz="1.0125000000000003e-08"/>
+        </inertial>
     </link>
     <joint name="back_yaw_joint" type="continuous">
-    <origin rpy="0 0 0" xyz="-0.120 0 -0.0775" />
-    <parent link="base_link" />
-    <child link="back_yaw_link" />
-    <axis xyz="0 0 1" />
-    <limit effort="${caster_effort_limit}" velocity="${caster_velocity_limit}" />
-    <dynamics damping="${caster_damping}" friction="${caster_friction}"/>
+        <origin rpy="0 0 0" xyz="-0.120 0 -0.0775" />
+        <parent link="base_link" />
+        <child link="back_yaw_link" />
+        <axis xyz="0 0 1" />
+        <limit effort="${caster_effort_limit}" velocity="${caster_velocity_limit}" />
+        <dynamics damping="${caster_damping}" friction="${caster_friction}"/>
     </joint>
     <link name="back_roll_link">
-    <visual>
-        <origin rpy="0 1.5707 1.5707" xyz="0 0 0"/>
-        <geometry>
-        <cylinder length="0.001" radius="0.0045000000000000005"/>
-        </geometry>
-        <material name="gray"/>
-    </visual>
-    <collision>
-        <origin rpy="0 1.5707 1.5707" xyz="0 0 0"/>
-        <geometry>
-        <cylinder length="0.001" radius="0.0045000000000000005"/>
-        </geometry>
-    </collision>
-    <inertial>
-        <origin rpy="0 1.5707 1.5707" xyz="0 0 0"/>
-        <mass value="0.001"/>
-        <inertia ixx="5.145833333333334e-09" ixy="0" ixz="0" iyy="5.145833333333334e-09" iyz="0" izz="1.0125000000000003e-08"/>
-    </inertial>
+        <visual>
+            <origin rpy="0 1.5707 1.5707" xyz="0 0 0"/>
+            <geometry>
+            <cylinder length="0.001" radius="0.0045000000000000005"/>
+            </geometry>
+            <material name="gray"/>
+        </visual>
+        <collision>
+            <origin rpy="0 1.5707 1.5707" xyz="0 0 0"/>
+            <geometry>
+            <cylinder length="0.001" radius="0.0045000000000000005"/>
+            </geometry>
+        </collision>
+        <inertial>
+            <origin rpy="0 1.5707 1.5707" xyz="0 0 0"/>
+            <mass value="0.001"/>
+            <inertia ixx="5.145833333333334e-09" ixy="0" ixz="0" iyy="5.145833333333334e-09" iyz="0" izz="1.0125000000000003e-08"/>
+        </inertial>
     </link>
     <joint name="back_roll_joint" type="continuous">
-    <origin rpy="0 0 0" xyz="0 0 0" />
-    <parent link="back_yaw_link" />
-    <child link="back_roll_link" />
-    <axis xyz="1 0 0" />
-    <limit effort="${caster_effort_limit}" velocity="${caster_velocity_limit}" />
-    <dynamics damping="${caster_damping}" friction="${caster_friction}"/>
+        <origin rpy="0 0 0" xyz="0 0 0" />
+        <parent link="back_yaw_link" />
+        <child link="back_roll_link" />
+        <axis xyz="1 0 0" />
+        <limit effort="${caster_effort_limit}" velocity="${caster_velocity_limit}" />
+        <dynamics damping="${caster_damping}" friction="${caster_friction}"/>
     </joint>
     <link name="back_pitch_link">
-    <visual>
-        <origin rpy="0 1.5707 1.5707" xyz="0 0 0"/>
-        <geometry>
-        <sphere radius="${caster_radius}"/>
-        </geometry>
-        <material name="gray"/>
-    </visual>
-    <collision>
-        <origin rpy="0 1.5707 1.5707" xyz="0 0 0"/>
-        <geometry>
-        <sphere radius="${caster_radius}"/>
-        </geometry>
-    </collision>
-    <inertial>
-        <origin rpy="0 1.5707 1.5707" xyz="0 0 0"/>
-        <mass value="${caster_mass}"/>
-        <inertia ixx="1.531733333333333e-05" ixy="0" ixz="0" iyy="1.531733333333333e-05" iyz="0" izz="1.531733333333333e-05"/>
-    </inertial>
-    </link>
-    <gazebo reference="back_pitch_link">
-        <kp>1000000000000000000000000000.0</kp>
-        <kd>1000000000000000000000000000.0</kd>
-        <mu1>0.5</mu1>
-        <mu2>0.5</mu2>
-        <material>Gazebo/Grey</material>
-    </gazebo>
+        <visual>
+            <origin rpy="0 1.5707 1.5707" xyz="0 0 0"/>
+            <geometry>
+            <sphere radius="${caster_radius}"/>
+            </geometry>
+            <material name="gray"/>
+        </visual>
+        <collision>
+            <origin rpy="0 1.5707 1.5707" xyz="0 0 0"/>
+            <geometry>
+            <sphere radius="${caster_radius}"/>
+            </geometry>
+        </collision>
+        <inertial>
+            <origin rpy="0 1.5707 1.5707" xyz="0 0 0"/>
+            <mass value="${caster_mass}"/>
+            <inertia ixx="1.531733333333333e-05" ixy="0" ixz="0" iyy="1.531733333333333e-05" iyz="0" izz="1.531733333333333e-05"/>
+        </inertial>
+    </link>
     <joint name="back_pitch_joint" type="continuous">
-    <origin rpy="0 0 0" xyz="0 0 0" />
-    <parent link="back_roll_link" />
-    <child link="back_pitch_link" />
-    <axis xyz="0 1 0" />
-    <limit effort="${caster_effort_limit}" velocity="${caster_velocity_limit}" />
-    <dynamics damping="${caster_damping}" friction="${caster_friction}"/>
-    </joint>
+        <origin rpy="0 0 0" xyz="0 0 0" />
+        <parent link="back_roll_link" />
+        <child link="back_pitch_link" />
+        <axis xyz="0 1 0" />
+        <limit effort="${caster_effort_limit}" velocity="${caster_velocity_limit}" />
+        <dynamics damping="${caster_damping}" friction="${caster_friction}"/>
+    </joint>
+   <!-- Standoff Rod 1 -->
     <xacro:standoff_rod rod_name="standoff_rod_1" />
-    <xacro:standoff_rod rod_name="standoff_rod_2" />
-    <xacro:standoff_rod rod_name="standoff_rod_3" />
-    <xacro:standoff_rod rod_name="standoff_rod_4" />
-    <gazebo reference="standoff_rod_1">
-        <material>Gazebo/Grey</material>
-    </gazebo>
     <joint name="joint_standoff_rod_1" type="fixed">
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
File: xacro/cup_holder_tray.xacro (robot description, xacro)
@@ -5,5 +5,5 @@
             <visual>
             <geometry>
-                <cylinder radius="${top_base_radius}" length="${top_base_length}"/>
+                <cylinder radius="${cup_holder_tray_radius}" length="${cup_holder_tray_length}"/>
             </geometry>
             <material name="green_dark"/>
@@ -12,10 +12,10 @@
             <origin rpy="0 0 0" xyz="0 0 0"/>
             <geometry>
-                <cylinder radius="${top_base_radius}" length="${top_base_length}"/>
+                <cylinder radius="${cup_holder_tray_radius}" length="${cup_holder_tray_length}"/>
             </geometry>
             </collision>
             <inertial>
             <origin rpy="0 0 0" xyz="0 0 0"/>
-            <mass value="${top_base_mass}"/>
+            <mass value="${cup_holder_tray_mass}"/>
             <inertia ixx="0.0028783333333333335" ixy="0" ixz="0" iyy="0.0028783333333333335" iyz="0" izz="0.00512"/>
             </inertial>
