Commit message: Added launch file that starts gazebo and spawns two robots (still need to change the name to rick and morty), and updated xacro files to add robot_name as parameter; gazebo and topics look as expected

File: xacro/barista_robot.gazebo.xacro (robot description, xacro)
@@ -49,8 +49,8 @@
         </gazebo>
         <!-- PLUGINS -->
-        <!-- JOINT PUBLISHER -->
         <gazebo>
             <plugin name="box_bot_joint_state" filename="libgazebo_ros_joint_state_publisher.so">
             <ros>
+                <namespace>/${robot_name}</namespace>
                 <remapping>~/out:=joint_states</remapping>
             </ros>
@@ -66,21 +66,26 @@
             </plugin>
         </gazebo>
-        <!-- Differential drive -->
         <gazebo>
             <plugin filename="libgazebo_ros_diff_drive.so" name="differential_drive_controller">
-            <!-- wheels -->
-            <left_joint>joint_left_wheel</left_joint>
-            <right_joint>joint_right_wheel</right_joint>
-            <!-- kinematics -->
-            <wheel_separation>0.1</wheel_separation>
-            <wheel_diameter>0.07</wheel_diameter>
-            <!-- limits -->
-            <max_wheel_torque>1.0</max_wheel_torque>
-            <max_wheel_acceleration>2.0</max_wheel_acceleration>
-            <!-- output -->
-            <publish_odom>true</publish_odom>
-            <publish_odom_tf>true</publish_odom_tf>
-            <odometry_frame>odom</odometry_frame>
-            <robot_base_frame>base_link</robot_base_frame>
+                <ros>
+                    <namespace>/${robot_name}</namespace>
+                    <remapping>/cmd_vel:=cmd_vel</remapping>
+                </ros>
+                <update_rate>100</update_rate>
+                <!-- Wheel joints -->
+                <left_joint>joint_left_wheel</left_joint>
+                <right_joint>joint_right_wheel</right_joint>
+                <!-- Kinematics -->
+                <wheel_separation>0.1</wheel_separation>
+                <wheel_diameter>0.07</wheel_diameter>
+                <publish_odom>true</publish_odom>
+                <!-- TF frames -->
+                <odometry_frame>${robot_name}/odom</odometry_frame>>
+                <robot_base_frame>${robot_name}/base_link</robot_base_frame>
+                <publish_odom_tf>true</publish_odom_tf>
+                <publish_wheel_tf>false</publish_wheel_tf>
+                <!-- Limits -->
+                <max_wheel_torque>1.0</max_wheel_torque>
+                <max_wheel_acceleration>2.0</max_wheel_acceleration>
             </plugin>
         </gazebo>
@@ -107,5 +112,5 @@
                 <plugin name="laser" filename="libgazebo_ros_ray_sensor.so">
                 <ros>
-                    <namespace></namespace>
+                    <namespace>/${robot_name}</namespace>
                     <remapping>~/out:=scan</remapping>
                 </ros>

File: xacro/barista_robot_model.urdf.xacro (robot description, xacro)
@@ -1,4 +1,5 @@
 <?xml version="1.0"?>
 <robot xmlns:xacro="http://www.ros.org/wiki/xacro" name="barista_robot">
+    <xacro:property name="robot_name" value="$(arg robot_name)"/>
     <xacro:include filename="$(find barista_robot_description)/xacro/barista_robot.gazebo.xacro" />
     <xacro:include filename="$(find barista_robot_description)/xacro/wheel.xacro" />

Commit message: Updated the colors of the robots in rviz and gazebo; blue for rick and red for morty

File: xacro/barista_robot.gazebo.xacro (robot description, xacro)
@@ -3,5 +3,10 @@
     <xacro:macro name="gazebo_elements">
         <gazebo reference="base_link">
-            <material>Gazebo/Green</material>
+            <xacro:if value="${robot_name == 'rick'}">
+                <material>Gazebo/Blue</material>
+            </xacro:if>
+            <xacro:if value="${robot_name == 'morty'}">
+                <material>Gazebo/Red</material>
+            </xacro:if>
         </gazebo>
         <gazebo reference="left_wheel">
@@ -46,5 +51,10 @@
         </gazebo>
         <gazebo reference="cup_holder_tray">
-            <material>Gazebo/Green</material>
+            <xacro:if value="${robot_name == 'rick'}">
+                <material>Gazebo/Blue</material>
+            </xacro:if>
+            <xacro:if value="${robot_name == 'morty'}">
+                <material>Gazebo/Red</material>
+            </xacro:if>
         </gazebo>
         <!-- PLUGINS -->

File: xacro/barista_robot_model.urdf.xacro (robot description, xacro)
@@ -30,6 +30,11 @@
     <xacro:property name="cup_holder_tray_z_offset" value="0.3425"/>
     <xacro:property name="include_laser" value="true"/>
-    <material name="green_dark">
-        <color rgba="0.0 0.5 0.0 1"/>
+    <xacro:property name="rick_color" value="0.0 0.0 0.5 1"/>
+    <xacro:property name="morty_color" value="0.5 0.0 0.0 1"/>
+    <material name="rick_material">
+        <color rgba="${rick_color}"/>
+    </material>
+    <material name="morty_material">
+        <color rgba="${morty_color}"/>
     </material>
     <material name="gray">
@@ -45,5 +50,5 @@
                 <cylinder radius="${base_radius}" length="${base_length}"/>
             </geometry>
-            <material name="green_dark"/>
+            <material name="${robot_name}_material"/>
         </visual>
         <collision>

File: xacro/cup_holder_tray.xacro (robot description, xacro)
@@ -7,5 +7,5 @@
                 <cylinder radius="${cup_holder_tray_radius}" length="${cup_holder_tray_length}"/>
             </geometry>
-            <material name="green_dark"/>
+            <material name="${robot_name}_material"/>
             </visual>
             <collision>
